Commit message: Added AI integration for the navigation and also

File: install/warehouse_robot_comp219/share/warehouse_robot_comp219/urdf/warehouse_robot.urdf.xacro (robot description, xacro)
@@ -1,157 +1 @@
-<?xml version="1.0"?>
-<robot name="warehouse_robot" xmlns:xacro="http://www.ros.org/wiki/xacro">
-  <!-- ── Properties ── -->
-  <xacro:property name="base_radius"  value="0.22"/>
-  <xacro:property name="base_height"  value="0.18"/>
-  <xacro:property name="wheel_radius" value="0.06"/>
-  <xacro:property name="wheel_width"  value="0.04"/>
-  <xacro:property name="wheel_sep"    value="0.28"/>
-  <xacro:property name="caster_r"     value="0.02"/>
-  <!-- BASE FOOTPRINT -->
-  <link name="base_footprint"/>
-  <joint name="base_footprint_joint" type="fixed">
-    <parent link="base_footprint"/>
-    <child  link="base_link"/>
-    <origin xyz="0 0 ${wheel_radius}" rpy="0 0 0"/>
-  </joint>
-  <!-- BASE LINK -->
-  <link name="base_link">
-    <visual>
-      <geometry><cylinder radius="${base_radius}" length="${base_height}"/></geometry>
-      <material name="blue"><color rgba="0.2 0.4 0.8 1"/></material>
-    </visual>
-    <collision>
-      <geometry><cylinder radius="${base_radius}" length="${base_height}"/></geometry>
-    </collision>
-    <inertial>
-      <mass value="10.0"/>
-      <inertia ixx="0.1" ixy="0" ixz="0" iyy="0.1" iyz="0" izz="0.18"/>
-    </inertial>
-  </link>
-  <!-- LEFT WHEEL -->
-  <link name="left_wheel">
-    <visual>
-      <geometry><cylinder radius="${wheel_radius}" length="${wheel_width}"/></geometry>
-      <material name="dark"><color rgba="0.1 0.1 0.1 1"/></material>
-    </visual>
-    <collision>
-      <geometry><cylinder radius="${wheel_radius}" length="${wheel_width}"/></geometry>
-    </collision>
-    <inertial>
-      <mass value="0.5"/>
-      <inertia ixx="0.001" ixy="0" ixz="0" iyy="0.001" iyz="0" izz="0.001"/>
-    </inertial>
-  </link>
-  <joint name="left_wheel_joint" type="continuous">
-    <parent link="base_link"/>
-    <child  link="left_wheel"/>
-    <origin xyz="0 ${wheel_sep} ${-base_height/2}" rpy="${pi/2} 0 0"/>
-    <axis xyz="0 0 1"/>
-  </joint>
-  <!-- RIGHT WHEEL -->
-  <link name="right_wheel">
-    <visual>
-      <geometry><cylinder radius="${wheel_radius}" length="${wheel_width}"/></geometry>
-      <material name="dark"/>
-    </visual>
-    <collision>
-      <geometry><cylinder radius="${wheel_radius}" length="${wheel_width}"/></geometry>
-    </collision>
-    <inertial>
-      <mass value="0.5"/>
-      <inertia ixx="0.001" ixy="0" ixz="0" iyy="0.001" iyz="0" izz="0.001"/>
-    </inertial>
-  </link>
-  <joint name="right_wheel_joint" type="continuous">
-    <parent link="base_link"/>
-    <child  link="right_wheel"/>
-    <origin xyz="0 ${-wheel_sep} ${-base_height/2}" rpy="${pi/2} 0 0"/>
-    <axis xyz="0 0 1"/>
-  </joint>
-  <!-- CASTER WHEEL -->
-  <link name="caster_wheel">
-    <visual>
-      <geometry><sphere radius="${caster_r}"/></geometry>
-      <material name="dark"/>
-    </visual>
-    <collision>
-      <geometry><sphere radius="${caster_r}"/></geometry>
-    </collision>
-    <inertial>
-      <mass value="0.1"/>
-      <inertia ixx="0.0001" ixy="0" ixz="0" iyy="0.0001" iyz="0" izz="0.0001"/>
-    </inertial>
-  </link>
-  <joint name="caster_joint" type="fixed">
-    <parent link="base_link"/>
-    <child  link="caster_wheel"/>
-    <origin xyz="${base_radius - caster_r} 0 ${-(base_height/2 + caster_r - wheel_radius)}" rpy="0 0 0"/>
-  </joint>
-  <!-- LIDAR LINK -->
-  <link name="lidar_link">
-    <visual>
-      <geometry><cylinder radius="0.04" length="0.06"/></geometry>
-      <material name="black"><color rgba="0.05 0.05 0.05 1"/></material>
-    </visual>
-    <collision>
-      <geometry><cylinder radius="0.04" length="0.06"/></geometry>
-    </collision>
-    <inertial>
-      <mass value="0.2"/>
-      <inertia ixx="0.0001" ixy="0" ixz="0" iyy="0.0001" iyz="0" izz="0.0001"/>
-    </inertial>
-  </link>
-  <joint name="lidar_joint" type="fixed">
-    <parent link="base_link"/>
-    <child  link="lidar_link"/>
-    <origin xyz="0 0 ${base_height/2 + 0.03}" rpy="0 0 0"/>
-  </joint>
-  <!-- GAZEBO: Differential drive plugin -->
-  <gazebo>
-    <plugin filename="gz-sim-diff-drive-system"
-            name="gz::sim::systems::DiffDrive">
-      <left_joint>left_wheel_joint</left_joint>
-      <right_joint>right_wheel_joint</right_joint>
-      <wheel_separation>${wheel_sep * 2}</wheel_separation>
-      <wheel_radius>${wheel_radius}</wheel_radius>
-      <odom_publish_frequency>20</odom_publish_frequency>
-      <topic>cmd_vel</topic>
-      <odom_topic>odom</odom_topic>
-      <frame_id>odom</frame_id>
-      <child_frame_id>base_footprint</child_frame_id>
-    </plugin>
-  </gazebo>
-  <!-- GAZEBO: Joint state publisher -->
-  <gazebo>
-    <plugin filename="gz-sim-joint-state-publisher-system"
-            name="gz::sim::systems::JointStatePublisher"/>
-  </gazebo>
-  <!-- GAZEBO: 2D LiDAR sensor -->
-  <gazebo reference="lidar_link">
-    <sensor name="lidar" type="gpu_lidar">
-      <update_rate>10</update_rate>
-      <topic>scan</topic>
-      <gz_frame_id>lidar_link</gz_frame_id>
-      <lidar>
-        <scan>
-          <horizontal>
-            <samples>360</samples>
-            <resolution>1</resolution>
-            <min_angle>-3.14159</min_angle>
-            <max_angle>3.14159</max_angle>
-          </horizontal>
-        </scan>
-        <range>
-          <min>0.12</min>
-          <max>10.0</max>
-          <resolution>0.01</resolution>
-        </range>
-        <noise>
-          <type>gaussian</type>
-          <mean>0.0</mean>
-          <stddev>0.01</stddev>
-        </noise>
-      </lidar>
-    </sensor>
-  </gazebo>
-</robot>
+/root/robot_project/urdf/warehouse_robot.urdf.xacro
